File: kicad/power_adapter/power_adapter.kicad_sch (KiCad schematic)
At the start: 9 parts, among them J1 Barrel_Jack, J2 Conn_01x03_Pin, Q1 PMV65XP,215, Q2 PMV65XP,215, U1 AMS1117-5.0

Commit message: Improving power adapter
Parts:
- C1: value 0.33uF -> 10uF
- C2: value 0.1uF -> 22uF; footprint Capacitor_SMD:C_0805_2012Metric -> Capacitor_Tantalum_SMD:CP_EIA-3528-21_Kemet-B; symbol Device:C_Small -> Device:C_Polarized_Small
Changed lines of the file:
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@@
     )
   )
-  (symbol (lib_id "Device:C_Small") (at 187.96 93.98 0) (unit 1)
+  (symbol (lib_id "Device:C_Polarized_Small") (at 187.96 93.98 0) (unit 1)
     (in_bom yes) (on_board yes) (dnp no) (fields_autoplaced)
-    (property "Reference" "C2" (at 190.5 92.7163 0)
+    (property "Reference" "C2" (at 190.5 92.1639 0)
       (effects (font (size 1.27 1.27)) (justify left))
     )
-    (property "Value" "0.1uF" (at 190.5 95.2563 0)
+    (property "Value" "22uF" (at 190.5 94.7039 0)
       (effects (font (size 1.27 1.27)) (justify left))
     )
-    (property "Footprint" "Capacitor_SMD:C_0805_2012Metric" (at 187.96 93.98 0)
+    (property "Footprint" "Capacitor_Tantalum_SMD:CP_EIA-3528-21_Kemet-B" (at 187.96 93.98 0)
       (effects (font (size 1.27 1.27)) hide)
     )
@@
       (effects (font (size 1.27 1.27)) (justify left))
     )
-    (property "Value" "0.33uF" (at 162.56 95.2563 0)
+    (property "Value" "10uF" (at 162.56 95.2563 0)
       (effects (font (size 1.27 1.27)) (justify left))
     )

Commit message: Power adapter fixes
Parts:
- D1: footprint Package_DIP:DIP-4_W7.62mm -> lib:Diode_Bridge_MBS
Connections:
- net at J1.1: now also D1.4; no longer D1.3
- net at J1.2: now also D1.3; no longer D1.4
Changed lines of the file:
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@@
     )
   )
-  (symbol (lib_id "Device:D_Bridge_+-AA") (at 118.11 87.63 0) (unit 1)
+  (symbol (lib_id "Device:D_Bridge_+-AA") (at 118.11 87.63 0) (mirror x) (unit 1)
     (in_bom yes) (on_board yes) (dnp no)
     (property "Reference" "D1" (at 118.11 87.63 0)
       (effects (font (size 1.27 1.27)))
     )
-    (property "Value" "D_Bridge_+-AA" (at 107.95 93.98 0)
+    (property "Value" "D_Bridge_+-AA" (at 107.95 81.28 0)
       (effects (font (size 1.27 1.27)))
     )
-    (property "Footprint" "Package_DIP:DIP-4_W7.62mm" (at 118.11 87.63 0)
+    (property "Footprint" "lib:Diode_Bridge_MBS" (at 118.11 87.63 0)
       (effects (font (size 1.27 1.27)) hide)
     )
